Commit message: fix: correct corrupted <collision> tag in elfin5.urdf.xacro
The opening tag was mangled to <collisi三>, causing
'xml.parsers.expat.ExpatError: mismatched tag: line 86' when moveit2 loads
the robot description via xacro.

File: references/src/elfin_robot/elfin5/elfin5_ros2_gazebo/urdf/elfin5.urdf.xacro (robot description, xacro)
@@ -65,5 +65,5 @@
       </material>
     </visual>
-    <collisi三>
+    <collision>
       <origin
         xyz="0 0 0"
